File: schematic/enlarger_timer.kicad_sch (KiCad schematic)
At the start: 60 parts, among them IC1 LD3985, J1 Screen, J2 LED, J3 5V, J4 ST-Link, J5 Start, J6 Switch_Light, SW1 Reset, SW2 But_Mem_Write, SW3 But_Mem_Read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

Commit message: Updated board: change button positions, add conneting holes
Connections:
- net But_BRI: now also U1.29 (PA4); no longer U1.25 (PA2)
- net But_TIM: now also U1.25 (PA2); no longer U1.29 (PA4)
Changed lines of the file:
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@@
     (effects (font (size 1.27 1.27)) (justify left bottom))
   )
-  (label "But_BRI" (at 140.97 39.37 0)
+  (label "But_TIM" (at 140.97 39.37 0)
     (effects (font (size 1.27 1.27)) (justify left bottom))
   )
@@
     (effects (font (size 1.27 1.27)) (justify left bottom))
   )
-  (label "But_TIM" (at 140.97 44.45 0)
+  (label "But_BRI" (at 140.97 44.45 0)
     (effects (font (size 1.27 1.27)) (justify left bottom))
   )
